Commit message: refine pose opt

File: self_topoexplore/data/urdf/turtlebot3_burger.urdf.xacro (robot description, xacro)
@@ -143,5 +143,5 @@
     <parent link="base_link"/>
     <child link="base_camera1"/>
-    <origin xyz="0.2 0 0.172" rpy="0 0 0"/>
+    <origin xyz="0.2 0 1" rpy="0 0 0"/>
   </joint>
   <link name="base_camera1">
@@ -150,5 +150,5 @@
     <parent link="base_link"/>
     <child link="base_camera2"/>
-    <origin xyz="0.0 0.1 0.172" rpy="0 0 1.57"/>
+    <origin xyz="0.0 0.1 1" rpy="0 0 1.57"/>
   </joint>
   <link name="base_camera2">
@@ -157,5 +157,5 @@
     <parent link="base_link"/>
     <child link="base_camera3"/>
-    <origin xyz="-0.2 0 0.172" rpy="0 0 3.14"/>
+    <origin xyz="-0.2 0 1" rpy="0 0 3.14"/>
   </joint>
   <link name="base_camera3">
@@ -164,5 +164,5 @@
     <parent link="base_link"/>
     <child link="base_camera4"/>
-    <origin xyz="0.0 -0.1 0.172" rpy="0 0 -1.57"/>
+    <origin xyz="0.0 -0.1 1" rpy="0 0 -1.57"/>
   </joint>
   <link name="base_camera4">

Commit message: finish relative pose estimation

File: self_topoexplore/data/urdf/turtlebot3_burger.urdf.xacro (robot description, xacro)
@@ -150,5 +150,5 @@
     <parent link="base_link"/>
     <child link="base_camera2"/>
-    <origin xyz="0.0 0.1 1" rpy="0 0 1.57"/>
+    <origin xyz="0.0 0.1 1" rpy="0 0 1.5707"/>
   </joint>
   <link name="base_camera2">
@@ -164,5 +164,5 @@
     <parent link="base_link"/>
     <child link="base_camera4"/>
-    <origin xyz="0.0 -0.1 1" rpy="0 0 -1.57"/>
+    <origin xyz="0.0 -0.1 1" rpy="0 0 -1.5707"/>
   </joint>
   <link name="base_camera4">
